Commit message: 1

File: hinson_ws/src/se5035/urdf/laser.urdf (robot description, URDF)
Before this commit: robot laser_test, 2 links, 1 joints
Links:
- removed link laser_link
- removed link map
- added link base_link
- added link laser_correct_link; visual cylinder length=0.05 radius=0.03
Joints:
- joint laser_link_joint: child laser_link -> laser_correct_link; origin xyz=0 0 0 -> xyz=0 0 0.2 rpy=0 0 0; parent map -> base_link
